Commit message: Make Robot ATV Sized

File: model/vehicle.xacro (robot description, xacro)
@@ -267,5 +267,5 @@
   <!-- Front Left Steering Joint -->
   <joint name="front_left_steering_joint" type="revolute">
-    <origin xyz="${wheel_offset} ${wheel_separation/2} -${wheel_radius/2}" rpy="0 0 0"/>
+    <origin xyz="${wheel_offset} ${wheel_separation/2} -${body_height/2.0}" rpy="0 0 0"/>
     <parent link="body_link"/>
     <child link="front_left_steering_link"/>
@@ -285,5 +285,5 @@
   <!-- Front Right Steering Joint -->
   <joint name="front_right_steering_joint" type="revolute">
-    <origin xyz="${wheel_offset} ${-wheel_separation/2} -${wheel_radius/2}" rpy="0 0 0"/>
+    <origin xyz="${wheel_offset} ${-wheel_separation/2} -${body_height/2.0}" rpy="0 0 0"/>
     <parent link="body_link"/>
     <child link="front_right_steering_link"/>
@@ -303,5 +303,5 @@
   <!-- Rear Left Wheel Joint -->
   <joint name="rear_left_wheel_joint" type="continuous">
-    <origin xyz="-${wheel_offset} ${wheel_separation/2} -${wheel_radius/2}" rpy="0 0 0"/>
+    <origin xyz="-${wheel_offset} ${wheel_separation/2} -${body_height/2.0}" rpy="0 0 0"/>
     <parent link="body_link"/>
     <child link="rear_left_wheel_link"/>
@@ -312,5 +312,5 @@
   <!-- Rear Right Wheel Joint -->
   <joint name="rear_right_wheel_joint" type="continuous">
-    <origin xyz="-${wheel_offset} ${-wheel_separation/2} -${wheel_radius/2}" rpy="0 0 0"/>
+    <origin xyz="-${wheel_offset} ${-wheel_separation/2} -${body_height/2.0}" rpy="0 0 0"/>
     <parent link="body_link"/>
     <child link="rear_right_wheel_link"/>

Commit message: Rename body_link to base_link

File: model/vehicle.xacro (robot description, xacro)
@@ -58,5 +58,5 @@
   <!-- Links -->
   <!-- Body Link -->
-  <link name="body_link">
+  <link name="base_link">
     <visual>
       <origin xyz="0.0 0.0 0.0" rpy="0.0 0.0 0.0"/>
@@ -268,5 +268,5 @@
   <joint name="front_left_steering_joint" type="revolute">
     <origin xyz="${wheel_offset} ${wheel_separation/2} -${body_height/2.0}" rpy="0 0 0"/>
-    <parent link="body_link"/>
+    <parent link="base_link"/>
     <child link="front_left_steering_link"/>
     <axis xyz="0 0 1"/>
@@ -286,5 +286,5 @@
   <joint name="front_right_steering_joint" type="revolute">
     <origin xyz="${wheel_offset} ${-wheel_separation/2} -${body_height/2.0}" rpy="0 0 0"/>
-    <parent link="body_link"/>
+    <parent link="base_link"/>
     <child link="front_right_steering_link"/>
     <axis xyz="0 0 1"/>
@@ -304,5 +304,5 @@
   <joint name="rear_left_wheel_joint" type="continuous">
     <origin xyz="-${wheel_offset} ${wheel_separation/2} -${body_height/2.0}" rpy="0 0 0"/>
-    <parent link="body_link"/>
+    <parent link="base_link"/>
     <child link="rear_left_wheel_link"/>
     <axis xyz="0 1 0"/>
@@ -313,5 +313,5 @@
   <joint name="rear_right_wheel_joint" type="continuous">
     <origin xyz="-${wheel_offset} ${-wheel_separation/2} -${body_height/2.0}" rpy="0 0 0"/>
-    <parent link="body_link"/>
+    <parent link="base_link"/>
     <child link="rear_right_wheel_link"/>
     <axis xyz="0 1 0"/>
@@ -323,5 +323,5 @@
     <axis xyz="0 1 0" />
     <origin xyz="${body_length/2 - camera_stick_size/2} ${camera_box_size/2 + camera_stick_size/2} ${camera_height/2}" rpy="0.0 0.0 0.0"/>
-    <parent link="body_link"/>
+    <parent link="base_link"/>
     <child link="camera_stick_link"/>
   </joint>
@@ -335,5 +335,5 @@
   </joint>
   <!-- Gazebo Parameters -->
-  <gazebo reference="body_link">
+  <gazebo reference="base_link">
     <mu1>0.0001</mu1>
     <mu2>0.0001</mu2>

Commit message: Change model and parameters for compatability

File: model/vehicle.xacro (robot description, xacro)
@@ -57,6 +57,9 @@
   <xacro:property name="max_wheel_angular_velocity" value="${max_velocity / wheel_radius}"/>
   <!-- Links -->
+  <!-- Base Link -->
+  <link name="base_link">
+  </link>
   <!-- Body Link -->
-  <link name="base_link">
+  <link name="body_link">
     <visual>
       <origin xyz="0.0 0.0 0.0" rpy="0.0 0.0 0.0"/>
@@ -265,8 +268,14 @@
   </link>
   <!-- Joints -->
+  <!-- Body to Base Joint -->
+  <joint name="body_to_base" type="fixed">
+      <origin xyz="0 0 ${body_height/2.0 + wheel_radius}" rpy="0 0 0"/>
+    <child link="body_link"/>
+    <parent link="base_link"/>
+  </joint>
   <!-- Front Left Steering Joint -->
   <joint name="front_left_steering_joint" type="revolute">
     <origin xyz="${wheel_offset} ${wheel_separation/2} -${body_height/2.0}" rpy="0 0 0"/>
-    <parent link="base_link"/>
+    <parent link="body_link"/>
     <child link="front_left_steering_link"/>
     <axis xyz="0 0 1"/>
@@ -286,5 +295,5 @@
   <joint name="front_right_steering_joint" type="revolute">
     <origin xyz="${wheel_offset} ${-wheel_separation/2} -${body_height/2.0}" rpy="0 0 0"/>
-    <parent link="base_link"/>
+    <parent link="body_link"/>
     <child link="front_right_steering_link"/>
     <axis xyz="0 0 1"/>
@@ -304,5 +313,5 @@
   <joint name="rear_left_wheel_joint" type="continuous">
     <origin xyz="-${wheel_offset} ${wheel_separation/2} -${body_height/2.0}" rpy="0 0 0"/>
-    <parent link="base_link"/>
+    <parent link="body_link"/>
     <child link="rear_left_wheel_link"/>
     <axis xyz="0 1 0"/>
@@ -313,5 +322,5 @@
   <joint name="rear_right_wheel_joint" type="continuous">
     <origin xyz="-${wheel_offset} ${-wheel_separation/2} -${body_height/2.0}" rpy="0 0 0"/>
-    <parent link="base_link"/>
+    <parent link="body_link"/>
     <child link="rear_right_wheel_link"/>
     <axis xyz="0 1 0"/>
@@ -323,5 +332,5 @@
     <axis xyz="0 1 0" />
     <origin xyz="${body_length/2 - camera_stick_size/2} ${camera_box_size/2 + camera_stick_size/2} ${camera_height/2}" rpy="0.0 0.0 0.0"/>
-    <parent link="base_link"/>
+    <parent link="body_link"/>
     <child link="camera_stick_link"/>
   </joint>
@@ -335,5 +344,5 @@
   </joint>
   <!-- Gazebo Parameters -->
-  <gazebo reference="base_link">
+  <gazebo reference="body_link">
     <mu1>0.0001</mu1>
     <mu2>0.0001</mu2>
